File: board/PicoCart.kicad_sch (KiCad schematic)
At the start: 29 parts, among them J1 MSX Bus (Odd-Even), J2 Micro_SD_Card, J3 UART, J4 DEBUG, J5 MSX Debug, J6 Pico Debug, J7 Ground Pins, J8 Ground Pins, J9 Edge Connector, U1 LD1117S33TR_SOT223, U2 74LS245, U3 74LS245, U4 74LS245, U5 74LS245, U6 Pico, U7 SN74LV1T34DBV

Commit message: Debug Board Design
Created a Debug board so that I can test the Main Pico logic against a
more controllable set of signals, rather than the MSX which provides a
very short window of usability
Parts:
- removed C6: 100nF, Capacitor_THT:C_Disc_D4.3mm_W1.9mm_P5.00mm, symbol Device:C
- removed J1: MSX Bus (Odd-Even), Connector_PinHeader_2.54mm:PinHeader_2x25_P2.54mm_Vertical, symbol Connector_Generic:Conn_02x25_Odd_Even
- removed J6: Pico Debug, Connector_PinHeader_2.54mm:PinHeader_2x10_P2.54mm_Vertical, symbol Connector_Generic:Conn_02x10_Counter_Clockwise
- removed J9: Edge Connector, Connector:MSX_Cartridge, symbol Connector_Generic:Conn_02x25_Odd_Even
- removed R1: 10K, Resistor_THT:R_Axial_DIN0204_L3.6mm_D1.6mm_P7.62mm_Horizontal, symbol Device:R
- removed RN1: 10K, Resistor_THT:R_Array_SIP5, symbol Device:R_Network04_Split
- removed U5: 74LS245, Package_DIP:DIP-20_W7.62mm, symbol 74xx:74LS245
- removed U7: SN74LV1T34DBV, Package_TO_SOT_SMD:SOT-23-5, symbol Logic_LevelTranslator:SN74LV1T34DBV
- added D1: LED, LED_THT:LED_D5.0mm, symbol Device:LED
- added J1: D_DEBUG, Connector_PinSocket_2.54mm:PinSocket_1x03_P2.54mm_Vertical, symbol Connector_Generic:Conn_01x03
- added J6: D_UART, Connector_PinSocket_2.54mm:PinSocket_1x03_P2.54mm_Vertical, symbol Connector_Generic:Conn_01x03
- added J9: DEBUG_I2C, Connector_PinHeader_2.54mm:PinHeader_1x04_P2.54mm_Vertical, symbol Connector_Generic:Conn_01x04
- added R1: R_Small, Resistor_THT:R_Axial_DIN0207_L6.3mm_D2.5mm_P15.24mm_Horizontal, symbol Device:R_Small
- added U8: Pico, Library:RPi_Pico_SMD_TH, symbol MCU_RaspberryPi_and_Boards:Pico
- U6: footprint MCU_RaspberryPi_and_Boards:RPi_Pico_SMD_TH -> Library:RPi_Pico_SMD_TH
Connections:
- net E_CLK is gone; now on net /I_CS1: J5.17 (Pin_17)
- net I_CLK is gone; now on net /I_WAIT: U6.31 (GPIO26_ADC0)
- net /E_CS1 is gone; now on net /I_READ: J5.24 (Pin_24)
- net /E_CS12 is gone; now on net /I_SLTSEL: J5.23 (Pin_23)
- net /E_CS2 is gone; now on net /DOE: J5.22 (Pin_22)
- net /E_READ is gone; now on net /I_CS2: J5.18 (Pin_18)
- net /E_SLTSEL is gone; now on net /DOUT: J5.21 (Pin_21)
- net /E_WRITE is gone; now on net /I_WAIT: J5.19 (Pin_19)
- net /WAIT is gone; now on net /AOE: J5.20 (Pin_20)
- net +3.3V: now also R1.1
- net +5V: now also J9.1 (Pin_1), U8.40 (VBUS)
- net E_A0: now also U4.2 (A0), U8.4 (GPIO2)
- net E_A1: now also U4.3 (A1), U8.5 (GPIO3)
- net E_A10: now also U8.16 (GPIO12)
- net E_A11: now also U8.17 (GPIO13)
- net E_A12: now also U8.19 (GPIO14)
- net E_A13: now also U8.20 (GPIO15)
- net E_A14: now also U8.21 (GPIO16)
- net E_A15: now also U8.22 (GPIO17)
- net E_A2: now also U4.4 (A2), U8.6 (GPIO4)
- net E_A3: now also U4.5 (A3), U8.7 (GPIO5)
- net E_A4: now also U4.6 (A4), U8.9 (GPIO6)
- net E_A5: now also U4.7 (A5), U8.10 (GPIO7)
- net E_A6: now also U4.8 (A6), U8.11 (GPIO8)
- net E_A7: now also U4.9 (A7), U8.12 (GPIO9)
- net E_A8: now also U8.14 (GPIO10)
- net E_A9: now also U8.15 (GPIO11)
- net GND: now also D1.1 (K), J1.2 (Pin_2), J6.3 (Pin_3), J9.2 (Pin_2), U8.13 (GND), U8.18 (GND), U8.23 (GND), U8.28 (GND), U8.3 (GND), U8.33 (AGND), U8.38 (GND), U8.42 (GND), U8.8 (GND)
- net /DOE: now also U6.27 (GPIO21); no longer U6.29 (GPIO22)
- net /DOUT: now also U6.29 (GPIO22); no longer U6.32 (GPIO27_ADC1)
- net /I_CS1: now also U8.25 (GPIO19)
- net /I_CS2: now also U8.26 (GPIO20)
- net /I_READ: now also U8.29 (GPIO22)
- net /I_SLTSEL: now also U8.34 (GPIO28_ADC2)
- net /I_WAIT: now also U8.24 (GPIO18); no longer U6.34 (GPIO28_ADC2)
- net /I_WRITE: now also J5.25 (Pin_25), U8.27 (GPIO21)
- net E_D0: no longer names the net of J5.32 (Pin_32)
- net E_D0: no longer U4.2 (A0)
- net E_D1: no longer names the net of J5.31 (Pin_31)
- net E_D1: no longer U4.3 (A1)
- net E_D2: no longer names the net of J5.30 (Pin_30)
- net E_D2: no longer U4.4 (A2)
- net E_D3: no longer names the net of J5.29 (Pin_29)
- net E_D3: no longer U4.5 (A3)
- net E_D4: no longer names the net of J5.28 (Pin_28)
- net E_D4: no longer U4.6 (A4)
- net E_D5: no longer names the net of J5.27 (Pin_27)
- net E_D5: no longer U4.7 (A5)
- net E_D6: no longer names the net of J5.26 (Pin_26)
- net E_D6: no longer U4.8 (A6)
- removed net E_D7: J5.25 (Pin_25), U4.9 (A7)
- net /AHOE renamed /AOE
- net /AOE: now also U3.19 (CE)
- removed net /ALOE: U3.19 (CE), U6.27 (GPIO21)
- net /I_CS12: no longer names the net of U6.7 (GPIO5)
- new net: J1.3 (Pin_3), U8.41 (SWCLK)
- new net: J1.1 (Pin_1), U8.43 (SWDIO)
- new net: D1.2 (A), R1.2
- new net D_UART_RX: J6.2 (Pin_2), U8.2 (GPIO1)
- new net D_UART_TX: J6.1 (Pin_1), U8.1 (GPIO0)
- new net SCL: J9.3 (Pin_3), U8.32 (GPIO27_ADC1)
- new net SDA: J9.4 (Pin_4), U8.31 (GPIO26_ADC0)
- no-connect marks 33 -> 21
Other:
- moved on the sheet: J7, J8
