File: boards/main_board/PicoCart.kicad_sch (KiCad schematic)
At the start: 29 parts, among them J1 MSX Bus (Odd-Even), J2 Micro_SD_Card, J3 UART, J4 DEBUG, J5 MSX Debug, J6 Pico Debug, J7 Ground Pins, J8 Ground Pins, J9 Edge Connector, U1 LD1117S33TR_SOT223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

Commit message: Added 16 data lines
Parts:
- removed J3: UART, Connector_PinSocket_2.54mm:PinSocket_1x03_P2.54mm_Vertical, symbol Connector_Generic:Conn_01x03
- added D1: D, Diode_THT:D_A-405_P7.62mm_Horizontal, symbol Device:D
- J4: footprint Connector_PinSocket_2.54mm:PinSocket_1x03_P2.54mm_Vertical -> Connector_JST:JST_PH_S3B-PH-K_1x03_P2.00mm_Horizontal
- U6: footprint RPi_Pico:RPi_Pico_SMD_TH -> PicoCartLibrary:RPi_Pico_SMD_TH
Connections:
- net UART_RX is gone; now on net I_D1: U6.2 (GPIO1)
- net UART_TX is gone; now on net I_D0: U6.1 (GPIO0)
- net +5V: now also D1.1 (K); no longer J9.45 (Pin_45), J9.47 (Pin_47)
- net E_CLK: no longer U5.8 (A6)
- net I_CLK: no longer U5.12 (B6), U6.31 (GPIO26_ADC0)
- net I_D0: no longer U2.18 (B0), U6.16 (GPIO12)
- net I_D1: no longer U2.17 (B1), U6.17 (GPIO13)
- net I_D2: now also U6.4 (GPIO2); no longer U2.16 (B2), U6.19 (GPIO14)
- net I_D3: now also U6.5 (GPIO3); no longer U2.15 (B3), U6.20 (GPIO15)
- net I_D4: now also U6.6 (GPIO4); no longer U2.14 (B4), U6.21 (GPIO16)
- net I_D5: now also U6.7 (GPIO5); no longer U2.13 (B5), U6.22 (GPIO17)
- net I_D6: now also U6.9 (GPIO6); no longer U2.12 (B6), U6.24 (GPIO18)
- net I_D7: now also U6.10 (GPIO7); no longer U2.11 (B7), U6.25 (GPIO19)
- net SPI_CS: now also U6.22 (GPIO17); no longer U6.12 (GPIO9)
- net SPI_MISO: now also U6.21 (GPIO16); no longer U6.11 (GPIO8)
- net SPI_MOSI: now also U6.25 (GPIO19); no longer U6.15 (GPIO11)
- net SPI_SCK: now also U6.24 (GPIO18); no longer U6.14 (GPIO10)
- net /AHOE: no longer RN1.2 (R1.2), U2.19 (CE), U6.26 (GPIO20)
- net /ALOE: no longer RN1.3 (R2.2), U3.19 (CE), U6.27 (GPIO21)
- net /DOE: now also U6.34 (GPIO28_ADC2); no longer U6.29 (GPIO22)
- net /DOUT: now also U6.29 (GPIO22); no longer U6.32 (GPIO27_ADC1)
- net /E_CS1: no longer U5.2 (A0)
- net /E_CS12: no longer U5.4 (A2)
- net /E_CS2: no longer U5.3 (A1)
- net /E_READ: now also U5.3 (A1); no longer U5.6 (A4)
- net /E_SLTSEL: now also U5.2 (A0); no longer U5.5 (A3)
- net /E_WRITE: now also U5.4 (A2); no longer U5.7 (A5)
- net /I_CS1: no longer U5.18 (B0), U6.5 (GPIO3)
- net /I_CS12: no longer U5.16 (B2), U6.7 (GPIO5)
- net /I_CS2: no longer U5.17 (B1), U6.6 (GPIO4)
- net /I_READ: now also U5.17 (B1); no longer U5.14 (B4), U6.9 (GPIO6)
- net /I_SLTSEL: now also U5.18 (B0), U6.27 (GPIO21); no longer U5.15 (B3), U6.4 (GPIO2)
- net /I_WAIT: now also U6.31 (GPIO26_ADC0); no longer U6.34 (GPIO28_ADC2)
- net /I_WRITE: now also U5.16 (B2), U6.26 (GPIO20); no longer U5.13 (B5), U6.10 (GPIO7)
- new net: D1.2 (A), J9.45 (Pin_45), J9.47 (Pin_47)
- new net I_D10: U2.16 (B2), U6.14 (GPIO10)
- new net I_D11: U2.15 (B3), U6.15 (GPIO11)
- new net I_D12: U2.14 (B4), U6.16 (GPIO12)
- new net I_D13: U2.13 (B5), U6.17 (GPIO13)
- new net I_D14: U2.12 (B6), U6.19 (GPIO14)
- new net I_D15: U2.11 (B7), U6.20 (GPIO15)
- new net I_D8: U2.18 (B0), U6.11 (GPIO8)
- new net I_D9: U2.17 (B1), U6.12 (GPIO9)
- new net /AOE: RN1.2 (R1.2), RN1.3 (R2.2), U2.19 (CE), U3.19 (CE), U6.32 (GPIO27_ADC1)
- no-connect marks 33 -> 41

Commit message: Change GPIO Pinout for 16-bit version
Other:
- note added: "/SLTSEL & /WRITE Can be used to determine direction"
Changed lines of the file:
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@@
+		)
+	)
+	(text "/SLTSEL & /WRITE Can be \nused to determine direction"
+		(exclude_from_sim yes)
+		(at 110.998 90.678 0)
+		(effects
+			(font
+				(size 1.27 1.27)
+			)
 		)
 	)
