File: boards/full_bus_board/PicoCart.kicad_sch (KiCad schematic)
At the start: 29 parts, among them J1 MSX Bus (Odd-Even), J2 Micro_SD_Card, J4 DEBUG, J5 MSX Debug, J6 Pico Debug, J7 Ground Pins, J8 Ground Pins, J9 Edge Connector, U1 LD1117S33TR_SOT223, U2 74LS245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

Commit message: Started PIO
Parts:
- removed unit 1 of RN1
- removed unit 2 of RN1
Connections:
- net GND: now also U2.19 (CE)
- net I_D0: no longer U3.18 (B0), U6.1 (GPIO0)
- net I_D1: no longer U3.17 (B1), U6.2 (GPIO1)
- net I_D2: no longer U3.16 (B2), U6.4 (GPIO2)
- net I_D3: no longer U3.15 (B3), U6.5 (GPIO3)
- net I_D4: no longer U3.14 (B4), U6.6 (GPIO4)
- net I_D5: no longer U3.13 (B5), U6.7 (GPIO5)
- net I_D6: no longer U3.12 (B6), U6.9 (GPIO6)
- net I_D7: no longer U3.11 (B7), U6.10 (GPIO7)
- net /AOE: no longer U2.19 (CE), U3.19 (CE)
- net /DOUT: now also U6.29 (GPIO22)
- net /I_READ: no longer U6.26 (GPIO20)
- net /I_WRITE: now also U6.26 (GPIO20); no longer U6.29 (GPIO22)
- net I_D10 renamed I_A10
- net I_D11 renamed I_A11
- net I_D12 renamed I_A12
- net I_D13 renamed I_A13
- net I_D14 renamed I_A14
- net I_D15 renamed I_A15
- net I_D8 renamed I_A8
- net I_D9 renamed I_A9
- new net I_A0: U3.18 (B0), U6.1 (GPIO0)
- new net I_A1: U3.17 (B1), U6.2 (GPIO1)
- new net I_A2: U3.16 (B2), U6.4 (GPIO2)
- new net I_A3: U3.15 (B3), U6.5 (GPIO3)
- new net I_A4: U3.14 (B4), U6.6 (GPIO4)
- new net I_A5: U3.13 (B5), U6.7 (GPIO5)
- new net I_A6: U3.12 (B6), U6.9 (GPIO6)
- new net I_A7: U3.11 (B7), U6.10 (GPIO7)
- no-connect marks 40 -> 41
